Commit message: modified parameters

File: src/m2wr_description/urdf/rover.xacro (robot description, xacro)
@@ -81,12 +81,12 @@
     <pose>0 0 0.1 0 0 0</pose>
     <inertial>
-      <mass value="2"/>
+      <mass value="2.5"/>
       <origin rpy="0 0 0" xyz="0 0 0"/>
-      <inertia ixx="0.001933" ixy="0" ixz="0" iyy="0.003533" iyz="0" izz="0.004933"/>
+      <inertia ixx="0.005020" ixy="0" ixz="0" iyy="0.01283" iyz="0" izz="0.017192"/>
     </inertial>
     <!-- body -->
     <collision name="collision_chassis">
       <geometry>
-        <box size="0.14 0.1 0.04"/>
+        <box size="0.245 0.15 0.04"/>
       </geometry>
     </collision>
@@ -94,152 +94,112 @@
       <origin rpy="0 0 0" xyz="0 0 0"/>
       <geometry>
-        <box size="0.14 0.1 0.04"/>
+        <box size="0.245 0.15 0.04"/>
       </geometry>
       <material name="blue"/>
     </visual>
-    <!-- front cylinder that holds the caster-->
-    <collision name="f_caster_wheel_hold">
-     <origin rpy=" 0 0 0" xyz="0.065 0 -0.025"/>
-      <geometry>
-        <cylinder length="0.0075" radius="0.0025"/>
-      </geometry>
-      <surface>
-        <friction>
-          <ode>
-            <mu>0</mu>
-            <mu2>0</mu2>
-            <slip1>0.0</slip1>
-            <slip2>0.0</slip2>
-          </ode>
-        </friction>
-      </surface>
-    </collision>
-    <visual>
-      <origin rpy="0 0 0" xyz="0.065 0 -0.025"/>
-      <geometry>
-        <cylinder length="0.0075" radius="0.0025"/>
-      </geometry>
-      <material name="blue"/>
-    </visual>
-    <!-- rear cylinder that holds the caster-->
-    <collision name="r_caster_wheel_hold">
-     <origin rpy=" 0 0 0" xyz="-0.065 0 -0.025"/>
-      <geometry>
-        <cylinder length="0.0075" radius="0.0025"/>
-      </geometry>
-      <surface>
-        <friction>
-          <ode>
-            <mu>0</mu>
-            <mu2>0</mu2>
-            <slip1>0.0</slip1>
-            <slip2>0.0</slip2>
-          </ode>
-        </friction>
-      </surface>
-    </collision>
-    <visual>
-      <origin rpy="0 0 0" xyz="-0.065 0 -0.025"/>
-      <geometry>
-        <cylinder length="0.0075" radius="0.0025"/>
-      </geometry>
-      <material name="blue"/>
-    </visual>
-    <!-- caster front -->
-    <collision name="caster_front_collision">
-      <origin rpy=" 0 0 0" xyz="0.065 0 -0.0275"/>
-      <geometry>
-        <sphere radius="0.00025"/>
-      </geometry>
-      <surface>
-        <friction>
-          <ode>
-            <mu>0</mu>
-            <mu2>0</mu2>
-            <slip1>0.0</slip1>
-            <slip2>0.0</slip2>
-          </ode>
-        </friction>
-      </surface>
-    </collision>
-    <visual name="caster_front_visual">
-      <origin rpy=" 0 0 0" xyz="0.065 0 -0.0275"/>
-      <geometry>
-        <sphere radius="0.00025"/>
-      </geometry>
-    </visual>
-    <!-- caster rear -->
-    <collision name="caster_rear_collision">
-      <origin rpy=" 0 0 0" xyz="-0.065 0.0 -0.0275"/>
-      <geometry>
-        <sphere radius="0.00025"/>
-      </geometry>
-      <surface>
-        <friction>
-          <ode>
-            <mu>0</mu>
-            <mu2>0</mu2>
-            <slip1>0.0</slip1>
-            <slip2>0.0</slip2>
-          </ode>
-        </friction>
-      </surface>
-    </collision>
-    <visual name="caster_rear_visual">
-      <origin rpy=" 0 0 0" xyz="-0.065 0.0 -0.0275"/>
-      <geometry>
-        <sphere radius="0.00025"/>
-      </geometry>
-    </visual>
-  </link>
-  <link name="link_right_wheel">
-    <inertial>
-      <mass value="0.5"/>
-      <origin rpy="0 1.5707 1.5707" xyz="0 0 0"/>
-      <inertia ixx="0.00012917" ixy="0" ixz="0" iyy="0.00012917" iyz="0" izz="0.000225"/>
-    </inertial>
-    <collision name="link_right_wheel_collision">
-      <origin rpy="0 1.5707 1.5707" xyz="0 0 0"/>
-      <geometry>
-        <cylinder length="0.015" radius="0.03"/>
-      </geometry>
-    </collision>
-    <visual name="link_right_wheel_visual">
-      <origin rpy="0 1.5707 1.5707" xyz="0 0 0"/>
-      <geometry>
-        <cylinder length="0.015" radius="0.03"/>
-      </geometry>
-    </visual>
-  </link>
-  <joint name="joint_right_wheel" type="continuous">
-    <origin rpy="0 0 0" xyz="0.01 -0.0575 0.0"/>
-    <child link="link_right_wheel"/>
-    <parent link="link_chassis"/>
-    <axis rpy="0 0 0" xyz="0 1 0"/>
-    <limit effort="5" velocity="10"/>
-    <joint_properties damping="0.0" friction="0.0"/>
-  </joint>
-  <link name="link_left_wheel">
-    <inertial>
-      <mass value="0.5"/>
-      <origin rpy="0 1.5707 1.5707" xyz="0 0 0"/>
-      <inertia ixx="0.00012917" ixy="0" ixz="0" iyy="0.00012917" iyz="0" izz="0.000225"/>
-    </inertial>
-    <collision name="link_left_wheel_collision">
-      <origin rpy="0 1.5707 1.5707" xyz="0 0 0"/>
-      <geometry>
-        <cylinder length="0.015" radius="0.03"/>
-      </geometry>
-    </collision>
-    <visual name="link_left_wheel_visual">
-      <origin rpy="0 1.5707 1.5707" xyz="0 0 0"/>
-      <geometry>
-        <cylinder length="0.015" radius="0.03"/>
-      </geometry>
-    </visual>
-  </link>
-  <joint name="joint_left_wheel" type="continuous">
-    <origin rpy="0 0 0" xyz="0.01 0.0575 0.0"/>
-    <child link="link_left_wheel"/>
+  </link>
+  <link name="right_front_wheel">
+    <inertial>
+      <mass value="0.5"/>
+      <origin rpy="0 1.5707 1.5707" xyz="0 0 0"/>
+      <inertia ixx="0.000306" ixy="0" ixz="0" iyy="0.0002312" iyz="0" izz="0.000306"/>
+    </inertial>
+    <collision name="right_front_wheel_collision">
+      <origin rpy="0 1.5707 1.5707" xyz="0 0 0"/>
+      <geometry>
+        <cylinder length="0.025" radius="0.035"/>
+      </geometry>
+    </collision>
+    <visual name="right_front_wheel_visual">
+      <origin rpy="0 1.5707 1.5707" xyz="0 0 0"/>
+      <geometry>
+        <cylinder length="0.025" radius="0.035"/>
+      </geometry>
+    </visual>
+  </link>
+  <joint name="right_front_wheel_joint" type="continuous">
+    <origin rpy="0 0 0" xyz="0.12 -0.0875 0.0"/>
+    <child link="right_front_wheel"/>
+    <parent link="link_chassis"/>
+    <axis rpy="0 0 0" xyz="0 1 0"/>
+    <limit effort="5" velocity="10"/>
+    <joint_properties damping="0.0" friction="0.0"/>
+  </joint>
+  <link name="right_back_wheel">
+    <inertial>
+      <mass value="0.5"/>
+      <origin rpy="0 1.5707 1.5707" xyz="0 0 0"/>
+      <inertia ixx="0.0002312" ixy="0" ixz="0" iyy="0.0002312" iyz="0" izz="0.000306"/>
+    </inertial>
+    <collision name="right_back_wheel_collision">
+      <origin rpy="0 1.5707 1.5707" xyz="0 0 0"/>
+      <geometry>
+        <cylinder length="0.025" radius="0.035"/>
+      </geometry>
+    </collision>
+    <visual name="right_back_wheel_visual">
+      <origin rpy="0 1.5707 1.5707" xyz="0 0 0"/>
+      <geometry>
+        <cylinder length="0.025" radius="0.035"/>
+      </geometry>
+    </visual>
+  </link>
+  <joint name="right_back_wheel_joint" type="continuous">
+    <origin rpy="0 0 0" xyz="-0.12 -0.0875 0.0"/>
+    <child link="right_back_wheel"/>
+    <parent link="link_chassis"/>
+    <axis rpy="0 0 0" xyz="0 1 0"/>
+    <limit effort="5" velocity="10"/>
+    <joint_properties damping="0.0" friction="0.0"/>
+  </joint>
+  <link name="left_front_wheel">
+    <inertial>
+      <mass value="0.5"/>
+      <origin rpy="0 1.5707 1.5707" xyz="0 0 0"/>
+      <inertia ixx="0.0002312" ixy="0" ixz="0" iyy="0.0002312" iyz="0" izz="0.000306"/>
+    </inertial>
+    <collision name="left_front_wheel_collision">
+      <origin rpy="0 1.5707 1.5707" xyz="0 0 0"/>
+      <geometry>
+        <cylinder length="0.025" radius="0.035"/>
+      </geometry>
+    </collision>
+    <visual name="left_front_wheel_visual">
+      <origin rpy="0 1.5707 1.5707" xyz="0 0 0"/>
+      <geometry>
+        <cylinder length="0.025" radius="0.035"/>
+      </geometry>
+    </visual>
+  </link>
+  <joint name="left_front_wheel" type="continuous">
+    <origin rpy="0 0 0" xyz="0.12 0.0875 0.0"/>
+    <child link="left_front_wheel"/>
+    <parent link="link_chassis"/>
+    <axis rpy="0 0 0" xyz="0 1 0"/>
+    <limit effort="5" velocity="10"/>
+    <joint_properties damping="0.0" friction="0.0"/>
+  </joint>
+  <link name="left_back_wheel">
+    <inertial>
+      <mass value="0.5"/>
+      <origin rpy="0 1.5707 1.5707" xyz="0 0 0"/>
+      <inertia ixx="0.0002312" ixy="0" ixz="0" iyy="0.0002312" iyz="0" izz="0.000306"/>
+    </inertial>
+    <collision name="left_back_wheel_collision">
+      <origin rpy="0 1.5707 1.5707" xyz="0 0 0"/>
+      <geometry>
+        <cylinder length="0.025" radius="0.035"/>
+      </geometry>
+    </collision>
+    <visual name="left_back_wheel_visual">
+      <origin rpy="0 1.5707 1.5707" xyz="0 0 0"/>
+      <geometry>
+        <cylinder length="0.025" radius="0.035"/>
+      </geometry>
+    </visual>
+  </link>
+  <joint name="left_back_wheel" type="continuous">
+    <origin rpy="0 0 0" xyz="-0.12 0.0875 0.0"/>
+    <child link="left_back_wheel"/>
     <parent link="link_chassis"/>
     <axis rpy="0 0 0" xyz="0 1 0"/>
@@ -268,25 +228,45 @@
   </link>
   <joint name="camera_joint" type="fixed">
-	    <origin xyz="0.085 0 0.05" rpy="0 1.0466 0"/>
+	    <origin xyz="0.13 0 0.065" rpy="0 1.0466 0"/>
 	    <child link="camera_link"/>
 	    <parent link="link_chassis"/>
             <axis rpy = "0 0 0" xyz="0 1 0" />
   </joint>
-  <transmission name = "joint_left_wheel_trans">
-  	<type> transmission_interface/SimpleTransmission </type>
-        <joint name = "joint_left_wheel">
-        	<hardwareInterface> hardware_interface/VelocityJointInterface </hardwareInterface>
-        </joint>
-        <actuator name = "joint_left_wheel_motor">
-                <hardwareInterface> hardware_interface/VelocityJointInterface </hardwareInterface>
-  		<mechanicalReduction>1</mechanicalReduction>
-	</actuator>
-  </transmission>
-  <transmission name = "joint_right_wheel_trans">
-  	<type> transmission_interface/SimpleTransmission </type>
-        <joint name = "joint_right_wheel">
-        	<hardwareInterface> hardware_interface/VelocityJointInterface </hardwareInterface>
-        </joint>
-        <actuator name = "joint_right_wheel_motor">
+  <transmission name = "left_back_wheel_trans">
+  	<type> transmission_interface/SimpleTransmission </type>
+        <joint name = "left_back_wheel">
+        	<hardwareInterface> hardware_interface/VelocityJointInterface </hardwareInterface>
+        </joint>
+        <actuator name = "left_back_wheel_motor">
+                <hardwareInterface> hardware_interface/VelocityJointInterface </hardwareInterface>
+  		<mechanicalReduction>1</mechanicalReduction>
+	</actuator>
+  </transmission>
+  <transmission name = "left_front_wheel_trans">
+  	<type> transmission_interface/SimpleTransmission </type>
+        <joint name = "left_front_wheel">
+        	<hardwareInterface> hardware_interface/VelocityJointInterface </hardwareInterface>
+        </joint>
+        <actuator name = "left_front_wheel_motor">
+                <hardwareInterface> hardware_interface/VelocityJointInterface </hardwareInterface>
+  		<mechanicalReduction>1</mechanicalReduction>
+	</actuator>
+  </transmission>
+  <transmission name = "right_back_wheel_trans">
+  	<type> transmission_interface/SimpleTransmission </type>
+        <joint name = "right_back_wheel">
+        	<hardwareInterface> hardware_interface/VelocityJointInterface </hardwareInterface>
+        </joint>
+        <actuator name = "right_back_wheel_motor">
+                <hardwareInterface> hardware_interface/VelocityJointInterface </hardwareInterface>
+  		<mechanicalReduction>1</mechanicalReduction>
+	</actuator>
+  </transmission>
+  <transmission name = "right_front_wheel_trans">
+  	<type> transmission_interface/SimpleTransmission </type>
+        <joint name = "right_front_wheel">
+        	<hardwareInterface> hardware_interface/VelocityJointInterface </hardwareInterface>
+        </joint>
+        <actuator name = "right_front_wheel_motor">
                 <hardwareInterface> hardware_interface/VelocityJointInterface </hardwareInterface>
   		<mechanicalReduction>1</mechanicalReduction>
@@ -296,4 +276,7 @@
   <plugin name="gazebo_ros_control" filename="libgazebo_ros_control.so">
     <robotNamespace>/rover</robotNamespace>
+    <controlPeriod>0.001</controlPeriod>
+    <robotSimType>gazebo_ros_control/DefaultRobotHWSim</robotSimType>
+    <legacyModeNS>true</legacyModeNS>
   </plugin>
 </gazebo>
